File: PCB/Quad0/Quad0.kicad_sch (KiCad schematic)
At the start: 96 parts, among them J1 DEBUG_CONN_PAD, J2 Mtype_Select, J3 Mtype_Select, J4 Mtype_Select, J5 Mtype_Select, J6 1N5819, J7 Power_Pad, Q1 DMN2024UFDF-7, Q2 DMN2024UFDF-7, Q3 DMN2024UFDF-7, Q4 DMN2024UFDF-7, SW1 RUN_BTN, SW2 BOOTSEL_BTN, U1 RP2350A_C42411118, U2 AP7361C-33E-13, U3 W25Q128JVSIQTR, U4 ABM8-272-T3_C20625731, U5 ICM-42688-P, U6 DPS368XTSA1, U7 BMM150, U8 ESP-01, U9 AP22818BKWT-7

Commit message: added footprints and jlc part numbers for main board
Parts:
- removed L1: 3.3u, symbol Device:L_Small
- added J10: GPIO[23-24], Connector_PinHeader_2.54mm:PinHeader_1x02_P2.54mm_Vertical, symbol Connector_Generic:Conn_01x02
- added J8: GPIO[18-22], Connector_PinHeader_2.54mm:PinHeader_1x05_P2.54mm_Vertical, symbol Connector_Generic:Conn_01x05
- added J9: GPIO[27-29], Connector_PinHeader_2.54mm:PinHeader_1x03_P2.54mm_Vertical, symbol Connector_Generic:Conn_01x03
- added L2: AOTA-B201610S3R3-101-T, easyeda2kicad:IND-SMD_L2.0-W1.6_AOTA-B201610S3R3-101-T, symbol easyeda2kicad:AOTA-B201610S3R3-101-T
- C1, C2, C32, C6: footprint (none) -> easyeda2kicad:C0603; LCSC Part (none) -> C19702; MPN (none) -> CL10A106KP8NNNC; Manufacturer (none) -> Samsung Electro-Mechanics
- C10, C11, C12, C13, C14, C15, C16, C17, C20, C21, C22, C23, C24, C25, C26, C27, C28, C29, C30, C31, C7, C8, C9: footprint (none) -> easyeda2kicad:C0402; LCSC Part (none) -> C1525; MPN (none) -> CL05B104KO5NNNC; Manufacturer (none) -> Samsung Electro-Mechanics
- C18, C19: footprint (none) -> easyeda2kicad:C0402; LCSC Part (none) -> C106997; MPN (none) -> CC0402JRNPO9BN150; Manufacturer (none) -> YAGEO
- C3, C4, C5: footprint (none) -> easyeda2kicad:C0402; LCSC Part (none) -> C77004; MPN (none) -> GRM155R61A475KEAAD; Manufacturer (none) -> Murata Electronics
- H1, H2, H3, H4: footprint (none) -> MountingHole:MountingHole_2mm
- J1: footprint (none) -> Connector_PinHeader_2.54mm:PinHeader_1x04_P2.54mm_Vertical
- J2, J3, J4, J5, J6, J7: footprint (none) -> Connector_PinHeader_2.54mm:PinHeader_1x02_P2.54mm_Vertical
- Motor1, Motor2, Motor3, Motor4: footprint (none) -> Connector_PinHeader_2.54mm:PinHeader_1x01_P2.54mm_Vertical
- R1, R2: footprint (none) -> easyeda2kicad:R0402; LCSC Part (none) -> C25905; MPN (none) -> 0402WGF5101TCE; Manufacturer (none) -> UNI-ROYAL(Uniroyal Elec)
- R10, R6, R8, R9: footprint (none) -> easyeda2kicad:R0402; LCSC Part (none) -> C11702; MPN (none) -> 0402WGF1001TCE; Manufacturer (none) -> UNI-ROYAL(Uniroyal Elec)
- R11, R13, R15, R17: footprint (none) -> easyeda2kicad:R0603; LCSC Part (none) -> C4275; MPN (none) -> 0603WAF750JT5E; Manufacturer (none) -> UNI-ROYAL(Uniroyal Elec)
- R12, R14, R16, R18, R21: footprint (none) -> easyeda2kicad:R0402; LCSC Part (none) -> C25741; MPN (none) -> 0402WGF1003TCE; Manufacturer (none) -> UNI-ROYAL(Uniroyal Elec)
- R19, R20: footprint (none) -> easyeda2kicad:R0402; LCSC Part (none) -> C25900; MPN (none) -> 0402WGF4701TCE; Manufacturer (none) -> UNI-ROYAL(Uniroyal Elec)
- R22, R23: footprint (none) -> easyeda2kicad:R0402; LCSC Part (none) -> C25079; MPN (none) -> 0402WGF1200TCE; Manufacturer (none) -> UNI-ROYAL(Uniroyal Elec)
- R24, R25: footprint (none) -> easyeda2kicad:R0402; LCSC Part (none) -> C25744; MPN (none) -> 0402WGF1002TCE; Manufacturer (none) -> UNI-ROYAL(Uniroyal Elec)
- R26: footprint (none) -> easyeda2kicad:R0402; LCSC Part (none) -> C25756; MPN (none) -> 0402WGF1502TCE; Manufacturer (none) -> UNI-ROYAL(Uniroyal Elec)
- R3: footprint (none) -> easyeda2kicad:R0402; LCSC Part (none) -> C25105; MPN (none) -> 0402WGF330JTCE; Manufacturer (none) -> UNI-ROYAL(Uniroyal Elec)
- R4, R5: footprint (none) -> easyeda2kicad:R0402; LCSC Part (none) -> C25100; MPN (none) -> 0402WGF270JTCE; Manufacturer (none) -> UNI-ROYAL(Uniroyal Elec)
Connections:
- net +1V1: now also L2.2
- net GPIO18: now also J8.1 (Pin_1)
- net GPIO19: now also J8.2 (Pin_2)
- net GPIO20: now also J8.3 (Pin_3)
- net GPIO21: now also J8.4 (Pin_4)
- net GPIO22: now also J8.5 (Pin_5)
- net GPIO23: now also J10.1 (Pin_1)
- net GPIO24: now also J10.2 (Pin_2)
- net GPIO27: now also J9.1 (Pin_1)
- net GPIO28: now also J9.2 (Pin_2)
- net GPIO29: now also J9.3 (Pin_3)
- net at U1.48 (VREG_LX): now also L2.1
- no-connect marks 20 -> 10

Commit message: pcb layout rev1
Parts:
- removed H4: MountingHole, MountingHole:MountingHole_2mm, symbol Mechanical:MountingHole
- Motor1, Motor2, Motor3, Motor4: footprint Connector_PinHeader_2.54mm:PinHeader_1x01_P2.54mm_Vertical -> Connector_PinHeader_2.54mm:PinHeader_1x02_P2.54mm_Vertical
Connections:
- net +BATT_Brushed: now also J6.2 (Pin_2), J7.1 (Pin_1), Motor1.1 (Pin_1), Motor2.1 (Pin_1), Motor3.1 (Pin_1), Motor4.1 (Pin_1); no longer J6.K (Pin_2), J7.PWR (Pin_1), Motor1.+ (Pin_1), Motor2.+ (Pin_1), Motor3.+ (Pin_1), Motor4.+ (Pin_1)
- net GND: now also J7.2 (Pin_2); no longer J7.GND (Pin_2)
- net USB_RAW_VBUS: now also J6.1 (Pin_1); no longer J6.A (Pin_1)
- net at R11.1: now also J4.2 (Pin_2); no longer J4.Sig (Pin_2)
- net at C23.2, D4.1 (A), Q4.1 (D)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: now also Motor4.2 (Pin_2); no longer Motor4.- (Pin_2)
- net at R13.1: now also J2.2 (Pin_2); no longer J2.Sig (Pin_2)
- net at C22.2, D3.1 (A), Q3.1 (D)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: now also Motor3.2 (Pin_2); no longer Motor3.- (Pin_2)
- net at C20.2, D1.1 (A), Q1.1 (D)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: now also Motor1.2 (Pin_2); no longer Motor1.- (Pin_2)
- net at R15.1: now also J3.2; no longer J3.Sig (Pin_2)
- net at C21.2, D2.1 (A), Q2.1 (D)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: now also Motor2.2 (Pin_2); no longer Motor2.- (Pin_2)
- net at R17.1: now also J5.2 (Pin_2); no longer J5.Sig (Pin_2)
Changed lines of the file:
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@@
 			)
 		)
-		(pin "PWR"
+		(pin "1"
 		)
-		(pin "GND"
+		(pin "2"
 		)
 		(instances
@@
 	)
 	(symbol
+		(lib_name "Conn_01x02_4")
 		(lib_id "Connector_Generic:Conn_01x02")
 		(at 453.39 170.18 270)
@@
 			)
 		)
-		(pin "Sig"
+		(pin "2"
 		)
 		(pin "1"
@@
 	)
 	(symbol
+		(lib_name "Conn_01x02_5")
 		(lib_id "Connector_Generic:Conn_01x02")
 		(at 379.73 170.18 270)
@@
 			)
 		)
-		(pin "Sig"
+		(pin "2"
 		)
 		(pin "1"
@@
 			)
 		)
-		(property "Footprint" "Connector_PinHeader_2.54mm:PinHeader_1x01_P2.54mm_Vertical"
+		(property "Footprint" "Connector_PinHeader_2.54mm:PinHeader_1x02_P2.54mm_Vertical"
 			(at 485.14 201.93 0)
 			(effects
@@
 			)
 		)
-		(pin "+"
+		(pin "2"
 		)
-		(pin "-"
+		(pin "1"
 		)
 		(instances
@@
 			)
 		)
-		(pin "K"
+		(pin "2"
 		)
-		(pin "A"
+		(pin "1"
 		)
 		(instances
@@
 			)
 		)
-		(pin "Sig"
+		(pin "2"
 		)
 		(pin "1"
@@
 	)
 	(symbol
-		(lib_id "Mechanical:MountingHole")
-		(at 128.27 265.43 0)
-		(unit 1)
-		(exclude_from_sim no)
-		(in_bom no)
-		(on_board yes)
-		(dnp no)
-		(fields_autoplaced yes)
-		(property "Reference" "H4"
-			(at 130.81 264.1599 0)
-			(effects
-				(font
-					(size 1.27 1.27)
-				)
-				(justify left)
-			)
-		)
-		(property "Value" "MountingHole"
-			(at 130.81 266.6999 0)
-			(effects
-				(font
-					(size 1.27 1.27)
-				)
-				(justify left)
-			)
-		)
-		(property "Footprint" "MountingHole:MountingHole_2mm"
-			(at 128.27 265.43 0)
-			(effects
-				(font
-					(size 1.27 1.27)
-				)
-				(hide yes)
-			)
-		)
-		(property "Datasheet" "~"
-			(at 128.27 265.43 0)
-			(effects
-				(font
-					(size 1.27 1.27)
-				)
-				(hide yes)
-			)
-		)
-		(property "Description" "Mounting Hole without connection"
-			(at 128.27 265.43 0)
-			(effects
-				(font
-					(size 1.27 1.27)
-				)
-				(hide yes)
-			)
-		)
-		(instances
-			(project "Quad0"
-				(path "/159302b8-19e4-4e7d-ac2c-4d85bb25e44b"
-					(reference "H4")
-					(unit 1)
-				)
-			)
-		)
-	)
-	(symbol
 		(lib_id "power:GND")
 		(at 335.28 105.41 0)
@@
 	)
 	(symbol
+		(lib_name "Conn_02x01_1")
 		(lib_id "Connector_Generic:Conn_02x01")
 		(at 485.14 157.48 270)
@@
 			)
 		)
-		(property "Footprint" "Connector_PinHeader_2.54mm:PinHeader_1x01_P2.54mm_Vertical"
+		(property "Footprint" "Connector_PinHeader_2.54mm:PinHeader_1x02_P2.54mm_Vertical"
 			(at 485.14 157.48 0)
 			(effects
@@
 			)
 		)
-		(pin "+"
+		(pin "2"
 		)
-		(pin "-"
+		(pin "1"
 		)
 		(instances
@@
 	)
 	(symbol
+		(lib_name "Conn_01x02_6")
 		(lib_id "Connector_Generic:Conn_01x02")
 		(at 379.73 214.63 270)
@@
 			)
 		)
-		(pin "Sig"
+		(pin "2"
 		)
 		(pin "1"
@@
 	)
 	(symbol
+		(lib_name "Conn_02x01_2")
 		(lib_id "Connector_Generic:Conn_02x01")
 		(at 411.48 157.48 270)
@@
 			)
 		)
-		(property "Footprint" "Connector_PinHeader_2.54mm:PinHeader_1x01_P2.54mm_Vertical"
+		(property "Footprint" "Connector_PinHeader_2.54mm:PinHeader_1x02_P2.54mm_Vertical"
 			(at 411.48 157.48 0)
 			(effects
@@
 			)
 		)
-		(pin "+"
+		(pin "2"
 		)
-		(pin "-"
+		(pin "1"
 		)
 		(instances
@@
 	)
 	(symbol
+		(lib_name "Conn_02x01_3")
 		(lib_id "Connector_Generic:Conn_02x01")
 		(at 411.48 201.93 270)
@@
 			)
 		)
-		(property "Footprint" "Connector_PinHeader_2.54mm:PinHeader_1x01_P2.54mm_Vertical"
+		(property "Footprint" "Connector_PinHeader_2.54mm:PinHeader_1x02_P2.54mm_Vertical"
 			(at 411.48 201.93 0)
 			(effects
@@
 			)
 		)
-		(pin "+"
+		(pin "2"
 		)
-		(pin "-"
+		(pin "1"
 		)
 		(instances

Commit message: pcb layout + routing v2
Parts:
- removed H3: MountingHole, MountingHole:MountingHole_2mm, symbol Mechanical:MountingHole
- removed J10: GPIO[23-24], Connector_PinHeader_2.54mm:PinHeader_1x02_P2.54mm_Vertical, symbol Connector_Generic:Conn_01x02
- added TP1: GPIO28_Pad, TestPoint:TestPoint_Pad_D1.0mm, symbol Connector:TestPoint
- added TP2: GPIO29_Pad, TestPoint:TestPoint_Pad_D1.0mm, symbol Connector:TestPoint
- J1: footprint Connector_PinHeader_2.54mm:PinHeader_1x04_P2.54mm_Vertical -> Connector_PinHeader_2.54mm:PinHeader_1x03_P2.54mm_Vertical; symbol Connector_Generic:Conn_01x05 -> Connector_Generic:Conn_01x03; now in the parts list
- J9: value GPIO[27-29] -> GPIO[23,24,27,28,29]; now in the parts list
Connections:
- net +BATT_Brushed: no longer USB1.A4B9 (VBUS)
- net GND: no longer J1.1 (Pin_1), J1.4 (Pin_4)
- net GPIO23: now also J9.1 (Pin_1)
- net GPIO24: now also J9.2 (Pin_2)
- net GPIO27: now also J9.3 (Pin_3); no longer J9.1 (Pin_1)
- net GPIO28: now also TP1.1; no longer J9.2 (Pin_2)
- net GPIO29: now also TP2.1; no longer J9.3 (Pin_3)
- net MCU_SWCLK: now also J1.3 (Pin_3); no longer J1.5 (Pin_5)
- net MCU_SWDIO: now also J1.1 (Pin_1); no longer J1.3 (Pin_3)
- net MCU_XOUT: now also U1.22 (XOUT)
- net USB_RAW_VBUS: now also USB1.A4B9 (VBUS)
- net USB_PICO-: now reaches R5.2, U1.51 (USB_DM)
- net USB_PICO+: now reaches R4.1, U1.52 (USB_DP)
Other:
- moved on the sheet: H1, H2

Commit message: pcb art + routing finished
Parts:
- added H3, H4: MountingHole, MountingHole:MountingHole_2mm, symbol Mechanical:MountingHole
Changed lines of the file:
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@@
 	)
 	(symbol
+		(lib_id "Mechanical:MountingHole")
+		(at 128.27 271.78 0)
+		(unit 1)
+		(exclude_from_sim no)
+		(in_bom no)
+		(on_board yes)
+		(dnp no)
+		(fields_autoplaced yes)
+		(property "Reference" "H4"
+			(at 130.81 270.5099 0)
+			(effects
+				(font
+					(size 1.27 1.27)
+				)
+				(justify left)
+			)
+		)
+		(property "Value" "MountingHole"
+			(at 130.81 273.0499 0)
+			(effects
+				(font
+					(size 1.27 1.27)
+				)
+				(justify left)
+			)
+		)
+		(property "Footprint" "MountingHole:MountingHole_2mm"
+			(at 128.27 271.78 0)
+			(effects
+				(font
+					(size 1.27 1.27)
+				)
+				(hide yes)
+			)
+		)
+		(property "Datasheet" "~"
+			(at 128.27 271.78 0)
+			(effects
+				(font
+					(size 1.27 1.27)
+				)
+				(hide yes)
+			)
+		)
+		(property "Description" "Mounting Hole without connection"
+			(at 128.27 271.78 0)
+			(effects
+				(font
+					(size 1.27 1.27)
+				)
+				(hide yes)
+			)
+		)
+		(instances
+			(project "Quad0"
+				(path "/159302b8-19e4-4e7d-ac2c-4d85bb25e44b"
+					(reference "H4")
+					(unit 1)
+				)
+			)
+		)
+	)
+	(symbol
 		(lib_id "power:GND")
 		(at 521.97 95.25 0)
@@
 					(unit 1)
 				)
+			)
+		)
+	)
+	(symbol
+		(lib_id "Mechanical:MountingHole")
+		(at 109.22 271.78 0)
+		(unit 1)
+		(exclude_from_sim no)
+		(in_bom no)
+		(on_board yes)
+		(dnp no)
+		(fields_autoplaced yes)
+		(property "Reference" "H3"
+			(at 111.76 270.5099 0)
+			(effects
+				(font
+					(size 1.27 1.27)
+				)
+				(justify left)
+			)
+		)
+		(property "Value" "MountingHole"
+			(at 111.76 273.0499 0)
+			(effects
+				(font
+					(size 1.27 1.27)
+				)
+				(justify left)
+			)
+		)
+		(property "Footprint" "MountingHole:MountingHole_2mm"
+			(at 109.22 271.78 0)
+			(effects
+				(font
+					(size 1.27 1.27)
+				)
+				(hide yes)
+			)
+		)
+		(property "Datasheet" "~"
+			(at 109.22 271.78 0)
+			(effects
+				(font
+					(size 1.27 1.27)
+				)
+				(hide yes)
+			)
+		)
+		(property "Description" "Mounting Hole without connection"
+			(at 109.22 271.78 0)
+			(effects
+				(font
+					(size 1.27 1.27)
+				)
+				(hide yes)
+			)
+		)
+		(instances
+			(project "Quad0"
+				(path "/159302b8-19e4-4e7d-ac2c-4d85bb25e44b"
+					(reference "H3")
+					(unit 1)
+				)
